Commit message: fix xacro

File: nachi_description/urdf/common.xacro (robot description, xacro)
@@ -1,4 +1,4 @@
 <?xml version="1.0"?>
-<robot>
-  <property name="M_PI" value="3.14159274"/>
+<robot xmlns:xacro="http://ros.org/wiki/xacro">
+  <xacro:property name="M_PI" value="3.14159274"/>
 </robot>

File: nachi_description/urdf/mz07/body.transmission.xacro (robot description, xacro)
@@ -4,14 +4,14 @@
 												 joint_name actuator_name
 												 reduction">
-	<transmission name="${name}">
-      <type>transmission_interface/SimpleTransmission</type>
-      <joint name="${joint_name}">
-		<hardwareInterface>PositionJointInterface</hardwareInterface>
-      </joint>
-      <actuator name="${actuator_name}">
-		<hardwareInterface>PositionJointInterface</hardwareInterface>
-		<mechanicalReduction>${reduction}</mechanicalReduction>
-      </actuator>
-	</transmission>
+      <transmission name="${name}">
+         <type>transmission_interface/SimpleTransmission</type>
+         <joint name="${joint_name}">
+            <hardwareInterface>hardware_interface/PositionJointInterface</hardwareInterface>
+         </joint>
+         <actuator name="${actuator_name}">
+            <hardwareInterface>hardware_interface/PositionJointInterface</hardwareInterface>
+            <mechanicalReduction>${reduction}</mechanicalReduction>
+         </actuator>
+      </transmission>
   </xacro:macro>
 </robot>
